File: Sunshine Sleep Mask PCB/Sunshine Sleep Mask PCB.kicad_sch (KiCad schematic)
At the start: 0 parts

Commit message: Adding Instructions
Parts:
- added BT1: Battery, symbol Device:Battery
- added J1, J4, J5: Conn_01x02_MountingPin, symbol Connector_Generic_MountingPin:Conn_01x02_MountingPin
- added J2, J3: Conn_01x04_MountingPin, symbol Connector_Generic_MountingPin:Conn_01x04_MountingPin
- added U1: ESP32-WROOM-32, RF_Module:ESP32-WROOM-32, symbol RF_Module:ESP32-WROOM-32
Connections:
- new net: U1.1 (GND), U1.15 (GND), U1.38 (GND), U1.39 (GND)

Commit message: Edits
Parts:
- removed J4: Conn_01x02_MountingPin, symbol Connector_Generic_MountingPin:Conn_01x02_MountingPin
- removed U1: ESP32-WROOM-32, RF_Module:ESP32-WROOM-32, symbol RF_Module:ESP32-WROOM-32
- added J4, J7: Conn_01x15_Socket, Connector_PinSocket_2.54mm:PinSocket_1x15_P2.54mm_Vertical, symbol Connector:Conn_01x15_Socket
- added J6: Connector_JST_Speaker_Left, Connector_JST:JST_PH_B2B-PH-K_1x02_P2.00mm_Vertical, symbol Connector_Generic_MountingPin:Conn_01x02_MountingPin
- added J8, J9: Conn_01x03_Pin, Connector_PinHeader_2.54mm:PinHeader_1x03_P2.54mm_Vertical, symbol Connector:Conn_01x03_Pin
- J1: value Conn_01x02_MountingPin -> Battery_JST_Connector; footprint (none) -> Connector_JST:JST_PH_B2B-PH-K_1x02_P2.00mm_Vertical
- J2: value Conn_01x04_MountingPin -> LED_JST_Connector_1; footprint (none) -> Connector_JST:JST_PH_B4B-PH-K_1x04_P2.00mm_Vertical
- J3: value Conn_01x04_MountingPin -> LED_JST_Connector_2; footprint (none) -> Connector_JST:JST_PH_B4B-PH-K_1x04_P2.00mm_Vertical
- J5: value Conn_01x02_MountingPin -> Connector_JST_Speaker_Right; footprint (none) -> Connector_JST:JST_PH_B2B-PH-K_1x02_P2.00mm_Vertical
Other:
- moved on the sheet: J1, J2, J5
