File: Sunshine Sleep Mask.kicad_sch (KiCad schematic)
At the start: 7 parts, among them J1 Conn_01x04, J2 Conn_01x02, J3 Conn_01x02, U2 ESP32-WROOM-32, U5 MAX98357A

Commit message: edited
Connections:
- new net: U3. (OUT-), U4. (OUT-)
Other:
- note added: "we did it"
Changed lines of the file:
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@@
+		)
+	)
+	(text "we did it"
+		(exclude_from_sim no)
+		(at 90.678 109.982 0)
+		(effects
+			(font
+				(size 1.27 1.27)
+			)
 		)
 	)
