File: Sunshine Sleep Mask PCB/0104-pcb/Adafruit MAX98357 Breakout.kicad_pcb (KiCad board)
At the start: 2 copper layers, 3 parts

Commit message: Clay 0408 Changes
Parts:
- JP1: footprint 1X07_ROUND_76 -> Audio_Module:1X07_ROUND_76
- U$10 (x2): footprint MOUNTINGHOLE_2.5_PLATED -> Audio_Module:MOUNTINGHOLE_2.5_PLATED
- moved U$10 0.29 mm to (179.7, 98.0)
